File: Cadlab_tester.kicad_pcb (KiCad board)
At the start: 2 copper layers, 30 x 30 mm, 3 parts, among them J1 Conn_01x02_Pin

Commit message: Rev2
Parts:
- added C1: 6n, Capacitor_SMD:C_1812_4532Metric, F.Cu at (129.9, 65.0)
- R1: value R -> 1k
- moved D1 2.96 mm to (121.0, 61.0)
- moved J1 0.15 mm to (126.5, 43.3)
Routing:
- net GND: track 21.0 -> 33.6 mm
- net Net-(D1-K): track 3.44 -> 15.1 mm
- net +3V3: track 21.3 -> 24.2 mm
Changed lines of the file:
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@@
   (net 3 "GND")
   (footprint "Connector_Molex:Molex_Micro-Fit_3.0_43650-0221_1x02_P3.00mm_Vertical" (layer "F.Cu")
-    (at 126.35 43.285)
+    (at 126.5 43.285)
     (descr "Molex Micro-Fit 3.0 Connector System, 43650-0221 (compatible alternatives: 43650-0222, 43650-0223), 2 Pins per row (https://www.molex.com/pdm_docs/sd/436500221_sd.pdf), generated with kicad-footprint-generator")
     (tags "connector Molex Micro-Fit_3.0 vertical")
@@
         (effects (font (size 1 1) (thickness 0.15)))
     )
-    (fp_text value "R" (at 0 2.2) (layer "F.Fab")
+    (fp_text value "1k" (at 0 2.2) (layer "F.Fab")
         (effects (font (size 1 1) (thickness 0.15)))
     )
@@
   )
   (footprint "LED_SMD:LED_2512_6332Metric" (layer "F.Cu")
-    (at 121 58 180)
+    (at 121 60.96 180)
     (descr "LED SMD 2512 (6332 Metric), square (rectangular) end terminal, IPC_7351 nominal, (Body size source: http://www.tortai-tech.com/upload/download/2011102023233369053.pdf), generated with kicad-footprint-generator")
     (tags "LED")
@@
     )
   )
+  (footprint "Capacitor_SMD:C_1812_4532Metric" (layer "F.Cu")
+    (at 129.95 65)
+    (descr "Capacitor SMD 1812 (4532 Metric), square (rectangular) end terminal, IPC_7351 nominal, (Body size source: IPC-SM-782 page 76, https://www.pcb-3d.com/wordpress/wp-content/uploads/ipc-sm-782a_amendment_1_and_2.pdf), generated with kicad-footprint-generator")
+    (tags "capacitor")
+    (property "Sheetfile" "Cadlab_tester.kicad_sch")
+    (property "Sheetname" "")
+    (property "ki_description" "Unpolarized capacitor")
+    (property "ki_keywords" "cap capacitor")
+    (attr smd)
+    (fp_text reference "C1" (at 0 -2.65) (layer "F.SilkS")
+        (effects (font (size 1 1) (thickness 0.15)))
+    )
+    (fp_text value "6n" (at 0 2.65) (layer "F.Fab")
+        (effects (font (size 1 1) (thickness 0.15)))
+    )
+    (fp_text user "${REFERENCE}" (at 0 0) (layer "F.Fab")
+        (effects (font (size 1 1) (thickness 0.15)))
+    )
+    (fp_line (start -1.161252 -1.71) (end 1.161252 -1.71)
+      (stroke (width 0.12) (type solid)) (layer "F.SilkS"))
+    (fp_line (start -1.161252 1.71) (end 1.161252 1.71)
+      (stroke (width 0.12) (type solid)) (layer "F.SilkS"))
+    (fp_line (start -3 -1.95) (end 3 -1.95)
+      (stroke (width 0.05) (type solid)) (layer "F.CrtYd"))
+    (fp_line (start -3 1.95) (end -3 -1.95)
+      (stroke (width 0.05) (type solid)) (layer "F.CrtYd"))
+    (fp_line (start 3 -1.95) (end 3 1.95)
+      (stroke (width 0.05) (type solid)) (layer "F.CrtYd"))
+    (fp_line (start 3 1.95) (end -3 1.95)
+      (stroke (width 0.05) (type solid)) (layer "F.CrtYd"))
+    (fp_line (start -2.25 -1.6) (end 2.25 -1.6)
+      (stroke (width 0.1) (type solid)) (layer "F.Fab"))
+    (fp_line (start -2.25 1.6) (end -2.25 -1.6)
+      (stroke (width 0.1) (type solid)) (layer "F.Fab"))
+    (fp_line (start 2.25 -1.6) (end 2.25 1.6)
+      (stroke (width 0.1) (type solid)) (layer "F.Fab"))
+    (fp_line (start 2.25 1.6) (end -2.25 1.6)
+      (stroke (width 0.1) (type solid)) (layer "F.Fab"))
+    (pad "1" smd roundrect (at -2.05 0) (size 1.4 3.4) (layers "F.Cu" "F.Paste" "F.Mask") (roundrect_rratio 0.178571)
+      (net 1 "Net-(D1-K)") (pintype "passive"))
+    (pad "2" smd roundrect (at 2.05 0) (size 1.4 3.4) (layers "F.Cu" "F.Paste" "F.Mask") (roundrect_rratio 0.178571)
+      (net 3 "GND") (pintype "passive"))
+    (model "${KICAD6_3DMODEL_DIR}/Capacitor_SMD.3dshapes/C_1812_4532Metric.wrl"
+      (offset (xyz 0 0 0))
+      (scale (xyz 1 1 1))
+      (rotate (xyz 0 0 0))
+    )
+  )
   (gr_line (start 110 70) (end 140 70)
     (stroke (width 0.1) (type default)) (layer "Edge.Cuts"))
@@
   (gr_line (start 140 40) (end 110 40)
     (stroke (width 0.1) (type default)) (layer "Edge.Cuts"))
-  (segment (start 124.32 57.58) (end 127.17 57.58) (width 0.25) (layer "F.Cu") (net 1))
-  (segment (start 123.9 58) (end 124.32 57.58) (width 0.25) (layer "F.Cu") (net 1))
-  (segment (start 118 58) (end 115 55) (width 0.25) (layer "F.Cu") (net 2))
-  (segment (start 115 49) (end 117.58 46.42) (width 0.25) (layer "F.Cu") (net 2))
-  (segment (start 118.1 58) (end 118 58) (width 0.25) (layer "F.Cu") (net 2))
-  (segment (start 115 55) (end 115 49) (width 0.25) (layer "F.Cu") (net 2))
-  (segment (start 117.58 46.42) (end 124.85 46.42) (width 0.25) (layer "F.Cu") (net 2))
+  (segment (start 123.9 60.96) (end 123.9 58.902) (width 0.25) (layer "F.Cu") (net 1))
+  (segment (start 123.9 58.902) (end 125.222 57.58) (width 0.25) (layer "F.Cu") (net 1))
+  (segment (start 125.222 63.5) (end 125.222 57.58) (width 0.25) (layer "F.Cu") (net 1))
+  (segment (start 125.222 57.58) (end 127.17 57.58) (width 0.25) (layer "F.Cu") (net 1))
+  (segment (start 126.722 65) (end 125.222 63.5) (width 0.25) (layer "F.Cu") (net 1))
+  (segment (start 127.9 65) (end 126.722 65) (width 0.25) (layer "F.Cu") (net 1))
+  (segment (start 115 55) (end 115 49) (width 0.5) (layer "F.Cu") (net 2))
+  (segment (start 117.58 46.42) (end 124.85 46.42) (width 0.5) (layer "F.Cu") (net 2))
+  (segment (start 118.1 60.96) (end 118.1 58.1) (width 0.5) (layer "F.Cu") (net 2))
+  (segment (start 118.1 58.1) (end 115 55) (width 0.5) (layer "F.Cu") (net 2))
+  (segment (start 115 49) (end 117.58 46.42) (width 0.5) (layer "F.Cu") (net 2))
   (segment (start 136 50) (end 133 50) (width 0.25) (layer "F.Cu") (net 3))
+  (segment (start 136.5 55.5) (end 137 55) (width 0.25) (layer "F.Cu") (net 3))
+  (segment (start 132 65) (end 134 65) (width 0.25) (layer "F.Cu") (net 3))
+  (segment (start 135 64) (end 135 57) (width 0.25) (layer "F.Cu") (net 3))
+  (segment (start 134.42 57.58) (end 136.5 55.5) (width 0.25) (layer "F.Cu") (net 3))
   (segment (start 137 55) (end 137 51) (width 0.25) (layer "F.Cu") (net 3))
   (segment (start 132.07 57.58) (end 134.42 57.58) (width 0.25) (layer "F.Cu") (net 3))
+  (segment (start 135 57) (end 136.5 55.5) (width 0.25) (layer "F.Cu") (net 3))
+  (segment (start 134 65) (end 135 64) (width 0.25) (layer "F.Cu") (net 3))
   (segment (start 129.42 46.42) (end 127.85 46.42) (width 0.25) (layer "F.Cu") (net 3))
   (segment (start 137 51) (end 136 50) (width 0.25) (layer "F.Cu") (net 3))
-  (segment (start 134.42 57.58) (end 137 55) (width 0.25) (layer "F.Cu") (net 3))
   (segment (start 133 50) (end 129.42 46.42) (width 0.25) (layer "F.Cu") (net 3))
 )
