File: Cadlab_tester.kicad_sch (KiCad schematic)
At the start: 3 parts, among them J1 Conn_01x02_Pin

Commit message: Schematico aggiornato
Parts:
- added C1: 6n, symbol Device:C
Connections:
- net GND: now also C1.2
- net at D1.1 (K), R1.1: now also C1.1
Other:
- moved on the sheet: J1
Changed lines of the file:
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@@
   (junction (at 115.57 73.66) (diameter 0) (color 0 0 0 0)
+  )
+  (junction (at 115.57 92.71) (diameter 0) (color 0 0 0 0)
+  )
+  (junction (at 129.54 100.33) (diameter 0) (color 0 0 0 0)
   )
   (junction (at 129.54 93.98) (diameter 0) (color 0 0 0 0)
@@
     (stroke (width 0) (type default))
   )
-  (wire (pts (xy 104.14 82.55) (xy 104.14 106.68))
+  (wire (pts (xy 104.14 86.36) (xy 104.14 107.95))
     (stroke (width 0) (type default))
   )
@@
     (stroke (width 0) (type default))
   )
-  (wire (pts (xy 97.79 80.01) (xy 110.49 80.01))
+  (wire (pts (xy 97.79 83.82) (xy 110.49 83.82))
     (stroke (width 0) (type default))
   )
@@
     (stroke (width 0) (type default))
   )
+  (wire (pts (xy 118.11 100.33) (xy 115.57 100.33))
+    (stroke (width 0) (type default))
+  )
+  (wire (pts (xy 115.57 100.33) (xy 115.57 92.71))
+    (stroke (width 0) (type default))
+  )
+  (wire (pts (xy 129.54 100.33) (xy 129.54 107.95))
+    (stroke (width 0) (type default))
+  )
   (wire (pts (xy 115.57 83.82) (xy 115.57 92.71))
     (stroke (width 0) (type default))
   )
-  (wire (pts (xy 97.79 82.55) (xy 104.14 82.55))
+  (wire (pts (xy 97.79 86.36) (xy 104.14 86.36))
+    (stroke (width 0) (type default))
+  )
+  (wire (pts (xy 125.73 100.33) (xy 129.54 100.33))
     (stroke (width 0) (type default))
   )
@@
     (stroke (width 0) (type default))
   )
-  (wire (pts (xy 110.49 80.01) (xy 110.49 73.66))
+  (wire (pts (xy 110.49 83.82) (xy 110.49 73.66))
     (stroke (width 0) (type default))
   )
-  (wire (pts (xy 104.14 106.68) (xy 129.54 106.68))
+  (wire (pts (xy 104.14 107.95) (xy 129.54 107.95))
     (stroke (width 0) (type default))
   )
@@
     (stroke (width 0) (type default))
   )
-  (wire (pts (xy 129.54 93.98) (xy 129.54 106.68))
+  (wire (pts (xy 129.54 93.98) (xy 129.54 100.33))
     (stroke (width 0) (type default))
   )
@@
     )
   )
+  (symbol (lib_id "Device:C") (at 121.92 100.33 90) (unit 1)
+    (in_bom yes) (on_board yes) (dnp no)
+    (property "Reference" "C1" (at 121.92 104.14 90)
+      (effects (font (size 1.27 1.27)))
+    )
+    (property "Value" "6n" (at 121.92 96.52 90)
+      (effects (font (size 1.27 1.27)))
+    )
+    (property "Footprint" "" (at 125.73 99.3648 0)
+      (effects (font (size 1.27 1.27)) hide)
+    )
+    (property "Datasheet" "~" (at 121.92 100.33 0)
+      (effects (font (size 1.27 1.27)) hide)
+    )
+    (pin "1")
+    (pin "2")
+    (instances
+      (project "Cadlab_tester"
+        (path "/cd5ceee6-a154-4203-98a0-7ff656fb7663"
+          (reference "C1") (unit 1)
+        )
+      )
+    )
+  )
   (symbol (lib_id "Device:R") (at 121.92 92.71 90) (unit 1)
     (in_bom yes) (on_board yes) (dnp no)
@@
     )
   )
-  (symbol (lib_id "Connector:Conn_01x02_Pin") (at 92.71 80.01 0) (unit 1)
+  (symbol (lib_id "Connector:Conn_01x02_Pin") (at 92.71 83.82 0) (unit 1)
     (in_bom yes) (on_board yes) (dnp no) (fields_autoplaced)
-    (property "Reference" "J1" (at 93.345 74.93 0)
+    (property "Reference" "J1" (at 93.345 78.74 0)
       (effects (font (size 1.27 1.27)))
     )
-    (property "Value" "Conn_01x02_Pin" (at 93.345 77.47 0)
+    (property "Value" "Conn_01x02_Pin" (at 93.345 81.28 0)
       (effects (font (size 1.27 1.27)))
     )
-    (property "Footprint" "Connector_Molex:Molex_Micro-Fit_3.0_43650-0221_1x02_P3.00mm_Vertical" (at 92.71 80.01 0)
+    (property "Footprint" "Connector_Molex:Molex_Micro-Fit_3.0_43650-0221_1x02_P3.00mm_Vertical" (at 92.71 83.82 0)
       (effects (font (size 1.27 1.27)) hide)
     )
-    (property "Datasheet" "~" (at 92.71 80.01 0)
+    (property "Datasheet" "~" (at 92.71 83.82 0)
       (effects (font (size 1.27 1.27)) hide)
     )

Commit message: Rev2
Parts:
- C1: footprint (none) -> Capacitor_SMD:C_1812_4532Metric
Changed lines of the file:
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@@
       (effects (font (size 1.27 1.27)))
     )
-    (property "Footprint" "" (at 125.73 99.3648 0)
+    (property "Footprint" "Capacitor_SMD:C_1812_4532Metric" (at 125.73 99.3648 0)
       (effects (font (size 1.27 1.27)) hide)
     )
